Commit message: reem_description: big update for hydro

File: reem_description/gazebo/gazebo.urdf.xacro (robot description, xacro)
@@ -1,5 +1,5 @@
 <?xml version="1.0"?>
 <!--
-  Copyright (c) 2011-2013, PAL Robotics, S.L.
+  Copyright (c) 2011-2014, PAL Robotics, S.L.
   All rights reserved.
   This work is licensed under the Creative Commons Attribution-NonCommercial-NoDerivs 3.0 Unported License.
@@ -11,5 +11,5 @@
        xmlns:interface="http://playerstage.sourceforge.net/gazebo/xmlschema/#interface">
   <gazebo>
-    <plugin filename="libros_control_gazebo_plugin.so" name="ros_control">
+    <plugin filename="libgazebo_ros_control.so" name="ros_control">
       <ns></ns>
       <robotSimType>reem_hardware_gazebo/ReemHardwareGazebo</robotSimType>

File: reem_description/robots/base.urdf.xacro (robot description, xacro)
@@ -1,5 +1,5 @@
 <?xml version="1.0"?>
 <!--
-  Copyright (c) 2012-2013, PAL Robotics, S.L.
+  Copyright (c) 2012-2014, PAL Robotics, S.L.
   All rights reserved.
   This work is licensed under the Creative Commons Attribution-NonCommercial-NoDerivs 3.0 Unported License.
@@ -14,9 +14,9 @@
   <!-- The following included files set up definitions of parts of the robot body -->
   <!-- Base -->
-  <include filename="$(find reem_description)/urdf/base/base.urdf.xacro" />
+  <xacro:include filename="$(find reem_description)/urdf/base/base.urdf.xacro" />
   <!-- Generic simulator_gazebo plugins -->
-<!--   <include filename="$(find reem_description)/gazebo/gazebo.urdf.xacro" /> -->
+<!--   <xacro:include filename="$(find reem_description)/gazebo/gazebo.urdf.xacro" /> -->
   <!-- Materials for visualization -->
-  <include filename="$(find reem_description)/urdf/materials.urdf.xacro" />
+  <xacro:include filename="$(find reem_description)/urdf/materials.urdf.xacro" />
   <!-- Base -->
   <xacro:reem_base  name="base"/>

File: reem_description/robots/reem_arm.urdf.xacro (robot description, xacro)
@@ -1,5 +1,5 @@
 <?xml version="1.0"?>
 <!--
-  Copyright (c) 2012-2013, PAL Robotics, S.L.
+  Copyright (c) 2012-2014, PAL Robotics, S.L.
   All rights reserved.
   This work is licensed under the Creative Commons Attribution-NonCommercial-NoDerivs 3.0 Unported License.
@@ -14,9 +14,9 @@
   <!-- The following included files set up definitions of parts of the robot body -->
   <!-- Arm -->
-  <include filename="$(find reem_description)/urdf/arm/arm.urdf.xacro" />
+  <xacro:include filename="$(find reem_description)/urdf/arm/arm.urdf.xacro" />
   <!-- Generic simulator_gazebo plugins -->
-  <include filename="$(find reem_description)/gazebo/gazebo.urdf.xacro" />
+  <xacro:include filename="$(find reem_description)/gazebo/gazebo.urdf.xacro" />
   <!-- Materials for visualization -->
-  <include filename="$(find reem_description)/urdf/materials.urdf.xacro" />
+  <xacro:include filename="$(find reem_description)/urdf/materials.urdf.xacro" />
   <!-- Fixed structure -->
   <joint name="base_footprint_joint" type="fixed">

File: reem_description/robots/reem_eye_hand_calibration_left_arm.urdf.xacro (robot description, xacro)
@@ -1,5 +1,5 @@
 <?xml version="1.0"?>
 <!--
-  Copyright (c) 2011-2013, PAL Robotics, S.L.
+  Copyright (c) 2011-2014, PAL Robotics, S.L.
   All rights reserved.
   This work is licensed under the Creative Commons Attribution-NonCommercial-NoDerivs 3.0 Unported License.
@@ -14,22 +14,22 @@
   <!-- The following included files set up definitions of parts of the robot body -->
   <!-- Base -->
-  <include filename="$(find reem_description)/urdf/base/base.urdf.xacro" />
+  <xacro:include filename="$(find reem_description)/urdf/base/base.urdf.xacro" />
   <!-- Torso -->
-  <include filename="$(find reem_description)/urdf/torso/torso.urdf.xacro" />
+  <xacro:include filename="$(find reem_description)/urdf/torso/torso.urdf.xacro" />
   <!-- Head -->
-  <include filename="$(find reem_description)/urdf/head/head.urdf.xacro" />
+  <xacro:include filename="$(find reem_description)/urdf/head/head.urdf.xacro" />
   <!-- Arm -->
-  <include filename="$(find reem_description)/urdf/arm/arm.urdf.xacro" />
+  <xacro:include filename="$(find reem_description)/urdf/arm/arm.urdf.xacro" />
   <!-- Hand -->
-  <include filename="$(find reem_description)/urdf/hand/hand.urdf.xacro" />
+  <xacro:include filename="$(find reem_description)/urdf/hand/hand.urdf.xacro" />
   <!-- Eye-hand calibration chessboard -->
-  <include filename="$(find reem_description)/urdf/eyeHandCalibrationChessBoard.urdf.xacro" />
+  <xacro:include filename="$(find reem_description)/urdf/eyeHandCalibrationChessBoard.urdf.xacro" />
   <!-- Camera sensors -->
-  <include filename="$(find reem_description)/urdf/sensors/stereo_camera.urdf.xacro" />
-<!--   <include filename="$(find reem_description)/urdf/sensors/back_camera.urdf.xacro" /> -->
+  <xacro:include filename="$(find reem_description)/urdf/sensors/stereo_camera.urdf.xacro" />
+<!--   <xacro:include filename="$(find reem_description)/urdf/sensors/back_camera.urdf.xacro" /> -->
   <!-- Generic simulator_gazebo plugins -->
-  <include filename="$(find reem_description)/gazebo/gazebo.urdf.xacro" />
+  <xacro:include filename="$(find reem_description)/gazebo/gazebo.urdf.xacro" />
   <!-- Materials for visualization -->
-  <include filename="$(find reem_description)/urdf/materials.urdf.xacro" />
+  <xacro:include filename="$(find reem_description)/urdf/materials.urdf.xacro" />
   <!-- Now we can start using the macros included above to define the actual robot -->
   <xacro:reem_base  name="base"/>

File: reem_description/robots/reem_eye_hand_calibration_right_arm.urdf.xacro (robot description, xacro)
@@ -1,5 +1,5 @@
 <?xml version="1.0"?>
 <!--
-  Copyright (c) 2011-2013, PAL Robotics, S.L.
+  Copyright (c) 2011-2014, PAL Robotics, S.L.
   All rights reserved.
   This work is licensed under the Creative Commons Attribution-NonCommercial-NoDerivs 3.0 Unported License.
@@ -14,22 +14,22 @@
   <!-- The following included files set up definitions of parts of the robot body -->
   <!-- Base -->
-  <include filename="$(find reem_description)/urdf/base/base.urdf.xacro" />
+  <xacro:include filename="$(find reem_description)/urdf/base/base.urdf.xacro" />
   <!-- Torso -->
-  <include filename="$(find reem_description)/urdf/torso/torso.urdf.xacro" />
+  <xacro:include filename="$(find reem_description)/urdf/torso/torso.urdf.xacro" />
   <!-- Head -->
-  <include filename="$(find reem_description)/urdf/head/head.urdf.xacro" />
+  <xacro:include filename="$(find reem_description)/urdf/head/head.urdf.xacro" />
   <!-- Arm -->
-  <include filename="$(find reem_description)/urdf/arm/arm.urdf.xacro" />
+  <xacro:include filename="$(find reem_description)/urdf/arm/arm.urdf.xacro" />
   <!-- Hand -->
-  <include filename="$(find reem_description)/urdf/hand/hand.urdf.xacro" />
+  <xacro:include filename="$(find reem_description)/urdf/hand/hand.urdf.xacro" />
   <!-- Eye-hand calibration chessboard -->
-  <include filename="$(find reem_description)/urdf/eyeHandCalibrationChessBoard.urdf.xacro" />
+  <xacro:include filename="$(find reem_description)/urdf/eyeHandCalibrationChessBoard.urdf.xacro" />
   <!-- Camera sensors -->
-  <include filename="$(find reem_description)/urdf/sensors/stereo_camera.urdf.xacro" />
-<!--   <include filename="$(find reem_description)/urdf/sensors/back_camera.urdf.xacro" /> -->
+  <xacro:include filename="$(find reem_description)/urdf/sensors/stereo_camera.urdf.xacro" />
+<!--   <xacro:include filename="$(find reem_description)/urdf/sensors/back_camera.urdf.xacro" /> -->
   <!-- Generic simulator_gazebo plugins -->
-  <include filename="$(find reem_description)/gazebo/gazebo.urdf.xacro" />
+  <xacro:include filename="$(find reem_description)/gazebo/gazebo.urdf.xacro" />
   <!-- Materials for visualization -->
-  <include filename="$(find reem_description)/urdf/materials.urdf.xacro" />
+  <xacro:include filename="$(find reem_description)/urdf/materials.urdf.xacro" />
   <!-- Now we can start using the macros included above to define the actual robot -->
   <xacro:reem_base  name="base"/>

File: reem_description/robots/reem_full.urdf.xacro (robot description, xacro)
@@ -1,5 +1,5 @@
 <?xml version="1.0"?>
 <!--
-  Copyright (c) 2011-2013, PAL Robotics, S.L.
+  Copyright (c) 2011-2014, PAL Robotics, S.L.
   All rights reserved.
   This work is licensed under the Creative Commons Attribution-NonCommercial-NoDerivs 3.0 Unported License.
@@ -14,23 +14,23 @@
   <!-- The following included files set up definitions of parts of the robot body -->
   <!-- Base -->
-  <include filename="$(find reem_description)/urdf/base/base.urdf.xacro" />
+  <xacro:include filename="$(find reem_description)/urdf/base/base.urdf.xacro" />
   <!-- Torso -->
-  <include filename="$(find reem_description)/urdf/torso/torso.urdf.xacro" />
+  <xacro:include filename="$(find reem_description)/urdf/torso/torso.urdf.xacro" />
   <!-- Head -->
-  <include filename="$(find reem_description)/urdf/head/head.urdf.xacro" />
+  <xacro:include filename="$(find reem_description)/urdf/head/head.urdf.xacro" />
   <!-- Arm -->
-  <include filename="$(find reem_description)/urdf/arm/arm.urdf.xacro" />
+  <xacro:include filename="$(find reem_description)/urdf/arm/arm.urdf.xacro" />
   <!-- Hand -->
-  <include filename="$(find reem_description)/urdf/hand/hand.urdf.xacro" />
+  <xacro:include filename="$(find reem_description)/urdf/hand/hand.urdf.xacro" />
   <!-- Camera sensors -->
-  <include filename="$(find reem_description)/urdf/sensors/stereo_camera.urdf.xacro" />
-  <include filename="$(find reem_description)/urdf/sensors/back_camera.urdf.xacro" />
+  <xacro:include filename="$(find reem_description)/urdf/sensors/stereo_camera.urdf.xacro" />
+  <xacro:include filename="$(find reem_description)/urdf/sensors/back_camera.urdf.xacro" />
   <!-- Generic simulator_gazebo plugins -->
-  <include filename="$(find reem_description)/gazebo/gazebo.urdf.xacro" />
+  <xacro:include filename="$(find reem_description)/gazebo/gazebo.urdf.xacro" />
   <!-- Materials for visualization -->
-  <include filename="$(find reem_description)/urdf/materials.urdf.xacro" />
+  <xacro:include filename="$(find reem_description)/urdf/materials.urdf.xacro" />
   <!-- Now we can start using the macros included above to define the actual robot -->
   <xacro:reem_base  name="base"/>
-  <xacro:reem_cargo  name="base"/>
+  <xacro:reem_cargo name="base"/>
   <xacro:reem_torso name="torso" parent="base_link"/>
   <xacro:reem_head  name="head"  parent="torso_2_link"/>
@@ -40,13 +40,13 @@
   <xacro:reem_hand name="hand" parent="arm_right_tool_link" side="right" reflect="1.0"  />
   <xacro:reem_hand name="hand" parent="arm_left_tool_link"  side="left"  reflect="-1.0" />
-  <include filename="$(find reem_description)/urdf/sensors/calibration.xacro"/>
+  <xacro:include filename="$(find reem_description)/urdf/sensors/calibration.xacro"/>
   <!-- stereo camera -->
   <!-- IMPORTANT: focal_length = image_width/(2tan(hfov/2)) -->
-  <xacro:stereo_camera_v0 parent="head_2_link" name="stereo" focal_length_left="459.838928" hfov_left="${71.0*deg_to_rad}" focal_length_right="459.838928" hfov_right="${71.0*deg_to_rad}" image_format="B8G8R8" image_width="656" image_height="492">
+  <xacro:stereo_camera_v0 parent="head_2_link" name="stereo" focal_length_left="459.840874" hfov_left="${71.0*deg_to_rad}" focal_length_right="459.840874" hfov_right="${71.0*deg_to_rad}" image_format="B8G8R8" image_width="656" image_height="492">
     <!-- The following transformations expresses the pose of the stereo_link (X pointing forward, Z upwards and Y leftwards, contrary to the stereo_optical_link which has Z pointing forward) wrt  head_2_link. -->
     <origin xyz="${cal_stereo_x} ${cal_stereo_y} ${cal_stereo_z}" rpy="${cal_stereo_roll} ${cal_stereo_pitch} ${cal_stereo_yaw}" />
   </xacro:stereo_camera_v0>
   <!-- back camera -->
-  <xacro:reem_back_camera parent="torso_2_link" name="back_camera" focal_length="376.003507" hfov="${89.999451423*deg_to_rad}" image_format="B8G8R8" image_width="752" image_height="480" >
+  <xacro:reem_back_camera parent="torso_2_link" name="back_camera" focal_length="376.002379" hfov="${89.999451423*deg_to_rad}" image_format="B8G8R8" image_width="752" image_height="480" >
     <!-- The following transformations expresses the pose of the back_camera_link (X pointing forward, Z upwards and Y leftwards) wrt torso_2_link. -->
     <!-- <origin xyz="-0.120 -0.302 -0.000" rpy="-3.142 1.571 0.211" /> -->

File: reem_description/robots/reem_head.urdf.xacro (robot description, xacro)
@@ -1,5 +1,5 @@
 <?xml version="1.0"?>
 <!--
-  Copyright (c) 2012-2013, PAL Robotics, S.L.
+  Copyright (c) 2012-2014, PAL Robotics, S.L.
   All rights reserved.
   This work is licensed under the Creative Commons Attribution-NonCommercial-NoDerivs 3.0 Unported License.
@@ -14,9 +14,9 @@
   <!-- The following included files set up definitions of parts of the robot body -->
   <!-- Head -->
-  <include filename="$(find reem_description)/urdf/head/head.urdf.xacro" />
+  <xacro:include filename="$(find reem_description)/urdf/head/head.urdf.xacro" />
   <!-- Generic simulator_gazebo plugins -->
-  <include filename="$(find reem_description)/gazebo/gazebo.urdf.xacro" />
+  <xacro:include filename="$(find reem_description)/gazebo/gazebo.urdf.xacro" />
   <!-- Materials for visualization -->
-  <include filename="$(find reem_description)/urdf/materials.urdf.xacro" />
+  <xacro:include filename="$(find reem_description)/urdf/materials.urdf.xacro" />
   <!-- Fixed structure -->
   <joint name="base_footprint_joint" type="fixed">

File: reem_description/robots/reem_rgbd.urdf.xacro (robot description, xacro)
@@ -1,5 +1,5 @@
 <?xml version="1.0"?>
 <!--
-  Copyright (c) 2013, PAL Robotics, S.L.
+  Copyright (c) 2013-2014, PAL Robotics, S.L.
   All rights reserved.
   This work is licensed under the Creative Commons Attribution-NonCommercial-NoDerivs 3.0 Unported License.
@@ -13,8 +13,9 @@
         name="reem" >
   <!-- Stock REEM robot -->
-  <include filename="$(find reem_description)/robots/reem_full.urdf.xacro" />
+  <xacro:include filename="$(find reem_description)/robots/reem_full.urdf.xacro" />
   <!-- Head-mounted ASUS Xtion Pro Live -->
-  <include filename="$(find reem_description)/urdf/sensors/xtion_pro_live.urdf.xacro" />
+  <xacro:include filename="$(find reem_description)/urdf/sensors/xtion_pro_live.urdf.xacro" />
   <xacro:xtion_pro_live parent="head_2_link" name="head_mount_xtion" > <!-- name is appended to create link and topic names -->
+     <!-- pose of head_mount_xtion_frame wrt /head_2_link -->
      <origin xyz="${cal_head_mount_xtion_x}
                   ${cal_head_mount_xtion_y}
@@ -23,4 +24,5 @@
                   ${cal_head_mount_xtion_pitch}
                   ${cal_head_mount_xtion_yaw}" />
+     <!-- pose of head_mount_xtion_optical_frame wrt head_mount_xtion_frame -->
      <origin xyz="0.0 0.0 0.0" rpy="-1.57 0.0 -1.57" />
 <!--

File: reem_description/robots/reem_right_hand_marker.urdf.xacro (robot description, xacro)
@@ -1,5 +1,5 @@
 <?xml version="1.0"?>
 <!--
-  Copyright (c) 2011-2013, PAL Robotics, S.L.
+  Copyright (c) 2011-2014, PAL Robotics, S.L.
   All rights reserved.
   This work is licensed under the Creative Commons Attribution-NonCommercial-NoDerivs 3.0 Unported License.
@@ -14,22 +14,22 @@
   <!-- The following included files set up definitions of parts of the robot body -->
   <!-- Base -->
-  <include filename="$(find reem_description)/urdf/base/base.urdf.xacro" />
+  <xacro:include filename="$(find reem_description)/urdf/base/base.urdf.xacro" />
   <!-- Torso -->
-  <include filename="$(find reem_description)/urdf/torso/torso.urdf.xacro" />
+  <xacro:include filename="$(find reem_description)/urdf/torso/torso.urdf.xacro" />
   <!-- Head -->
-  <include filename="$(find reem_description)/urdf/head/head.urdf.xacro" />
+  <xacro:include filename="$(find reem_description)/urdf/head/head.urdf.xacro" />
   <!-- Arm -->
-  <include filename="$(find reem_description)/urdf/arm/arm.urdf.xacro" />
+  <xacro:include filename="$(find reem_description)/urdf/arm/arm.urdf.xacro" />
   <!-- Hand -->
-  <include filename="$(find reem_description)/urdf/hand/hand.urdf.xacro" />
+  <xacro:include filename="$(find reem_description)/urdf/hand/hand.urdf.xacro" />
   <!-- Hand Marker-->
-  <include filename="$(find reem_description)/urdf/marker/marker.urdf.xacro" />
+  <xacro:include filename="$(find reem_description)/urdf/marker/marker.urdf.xacro" />
   <!-- Camera sensors -->
-  <include filename="$(find reem_description)/urdf/sensors/stereo_camera.urdf.xacro" />
-  <include filename="$(find reem_description)/urdf/sensors/back_camera.urdf.xacro" />
+  <xacro:include filename="$(find reem_description)/urdf/sensors/stereo_camera.urdf.xacro" />
+  <xacro:include filename="$(find reem_description)/urdf/sensors/back_camera.urdf.xacro" />
   <!-- Generic simulator_gazebo plugins -->
-  <include filename="$(find reem_description)/gazebo/gazebo.urdf.xacro" />
+  <xacro:include filename="$(find reem_description)/gazebo/gazebo.urdf.xacro" />
   <!-- Materials for visualization -->
-  <include filename="$(find reem_description)/urdf/materials.urdf.xacro" />
+  <xacro:include filename="$(find reem_description)/urdf/materials.urdf.xacro" />
   <!-- Now we can start using the macros included above to define the actual robot -->
   <xacro:reem_base  name="base"/>
@@ -45,10 +45,10 @@
   <!-- stereo camera -->
   <!-- IMPORTANT: focal_length = image_width/(2tan(hfov/2)) Ex.: f=359.000019  hfov=84.832707076 -->
-  <xacro:stereo_camera_v0 parent="head_2_link" name="stereo" focal_length_left="459.838928" hfov_left="${71.0*deg_to_rad}" focal_length_right="459.838928" hfov_right="${71.0*deg_to_rad}" image_format="B8G8R8" image_width="656" image_height="492">
+  <xacro:stereo_camera_v0 parent="head_2_link" name="stereo" focal_length_left="459.840874" hfov_left="${71.0*deg_to_rad}" focal_length_right="459.840874" hfov_right="${71.0*deg_to_rad}" image_format="B8G8R8" image_width="656" image_height="492">
     <!-- The following transformations expresses the pose of the stereo_link (X pointing forward, Z upwards and Y leftwards, contrary to the stereo_optical_link which has Z pointing forward) wrt  head_2_link. -->
     <!-- <origin xyz="0.0558343 -0.106811 0.0254842" rpy="1.61 -0.00976311 -0.0519005" /> -->
     <origin xyz="0.0558343 -0.106811 0.0365" rpy="1.5707 0 0" /> <!-- PERFECT SIMULATION -->
   </xacro:stereo_camera_v0>
-  <xacro:reem_back_camera parent="torso_2_link" name="back_camera" focal_length="376.003507" hfov="${89.999451423*deg_to_rad}" image_format="B8G8R8" image_width="752" image_height="480" >
+  <xacro:reem_back_camera parent="torso_2_link" name="back_camera" focal_length="376.002379" hfov="${89.999451423*deg_to_rad}" image_format="B8G8R8" image_width="752" image_height="480" >
     <!-- The following transformations expresses the pose of the back_camera_link (X pointing forward, Z upwards and Y leftwards) wrt torso_2_link. -->
     <!-- <origin xyz="-0.120 -0.302 -0.000" rpy="-3.142 1.571 0.211" /> -->

File: reem_description/robots/reem_torso.urdf.xacro (robot description, xacro)
@@ -1,5 +1,5 @@
 <?xml version="1.0"?>
 <!--
-  Copyright (c) 2012-2013, PAL Robotics, S.L.
+  Copyright (c) 2012-2014, PAL Robotics, S.L.
   All rights reserved.
   This work is licensed under the Creative Commons Attribution-NonCommercial-NoDerivs 3.0 Unported License.
@@ -14,9 +14,9 @@
   <!-- The following included files set up definitions of parts of the robot body -->
   <!-- Torso -->
-  <include filename="$(find reem_description)/urdf/torso/torso.urdf.xacro" />
+  <xacro:include filename="$(find reem_description)/urdf/torso/torso.urdf.xacro" />
   <!-- Generic simulator_gazebo plugins -->
-  <include filename="$(find reem_description)/gazebo/gazebo.urdf.xacro" />
+  <xacro:include filename="$(find reem_description)/gazebo/gazebo.urdf.xacro" />
   <!-- Materials for visualization -->
-  <include filename="$(find reem_description)/urdf/materials.urdf.xacro" />
+  <xacro:include filename="$(find reem_description)/urdf/materials.urdf.xacro" />
   <link name="base_footprint">
     <inertial>

File: reem_description/robots/reem_upper_body.urdf.xacro (robot description, xacro)
@@ -1,5 +1,5 @@
 <?xml version="1.0"?>
 <!--
-  Copyright (c) 2012-2013, PAL Robotics, S.L.
+  Copyright (c) 2012-2014, PAL Robotics, S.L.
   All rights reserved.
   This work is licensed under the Creative Commons Attribution-NonCommercial-NoDerivs 3.0 Unported License.
@@ -14,15 +14,15 @@
   <!-- The following included files set up definitions of parts of the robot body -->
   <!-- Torso -->
-  <include filename="$(find reem_description)/urdf/torso/torso.urdf.xacro" />
+  <xacro:include filename="$(find reem_description)/urdf/torso/torso.urdf.xacro" />
   <!-- Head -->
-  <include filename="$(find reem_description)/urdf/head/head.urdf.xacro" />
+  <xacro:include filename="$(find reem_description)/urdf/head/head.urdf.xacro" />
   <!-- Arm -->
-  <include filename="$(find reem_description)/urdf/arm/arm.urdf.xacro" />
+  <xacro:include filename="$(find reem_description)/urdf/arm/arm.urdf.xacro" />
   <!-- Hand -->
-  <include filename="$(find reem_description)/urdf/hand/hand.urdf.xacro" />
+  <xacro:include filename="$(find reem_description)/urdf/hand/hand.urdf.xacro" />
   <!-- Generic simulator_gazebo plugins -->
-  <include filename="$(find reem_description)/gazebo/gazebo.urdf.xacro" />
+  <xacro:include filename="$(find reem_description)/gazebo/gazebo.urdf.xacro" />
   <!-- Materials for visualization -->
-  <include filename="$(find reem_description)/urdf/materials.urdf.xacro" />
+  <xacro:include filename="$(find reem_description)/urdf/materials.urdf.xacro" />
   <link name="base_link">
     <inertial>

File: reem_description/robots/reem_with_xtion_link.urdf.xacro (robot description, xacro)
@@ -1,5 +1,5 @@
 <?xml version="1.0"?>
 <!--
-  Copyright (c) 2013, PAL Robotics, S.L.
+  Copyright (c) 2013-2014, PAL Robotics, S.L.
   All rights reserved.
   This work is licensed under the Creative Commons Attribution-NonCommercial-NoDerivs 3.0 Unported License.
@@ -13,5 +13,5 @@
         name="reem" >
   <!-- Stock REEM robot -->
-  <include filename="$(find reem_description)/robots/reem_full.urdf.xacro" />
+  <xacro:include filename="$(find reem_description)/robots/reem_full.urdf.xacro" />
   <!-- PAL printed xtion mount link on top of the head -->
   <joint name="head_mount_xtion_joint" type="fixed">
