Commit message: reem_description: big update for hydro

File: reem_description/robots/reem_wrist.urdf.xacro (robot description, xacro)
@@ -1,5 +1,5 @@
 <?xml version="1.0"?>
 <!--
-  Copyright (c) 2012-2013, PAL Robotics, S.L.
+  Copyright (c) 2012-2014, PAL Robotics, S.L.
   All rights reserved.
   This work is licensed under the Creative Commons Attribution-NonCommercial-NoDerivs 3.0 Unported License.
@@ -14,9 +14,9 @@
   <!-- The following included files set up definitions of parts of the robot body -->
   <!-- Wrist -->
-  <include filename="$(find reem_description)/urdf/arm/wrist.urdf.xacro" />
+  <xacro:include filename="$(find reem_description)/urdf/arm/wrist.urdf.xacro" />
   <!-- Generic simulator_gazebo plugins -->
-  <include filename="$(find reem_description)/gazebo/gazebo.urdf.xacro" />
+  <xacro:include filename="$(find reem_description)/gazebo/gazebo.urdf.xacro" />
   <!-- Materials for visualization -->
-  <include filename="$(find reem_description)/urdf/materials.urdf.xacro" />
+  <xacro:include filename="$(find reem_description)/urdf/materials.urdf.xacro" />
   <!-- Fixed structure -->
   <joint name="base_footprint_joint" type="fixed">

File: reem_description/urdf/arm/arm.transmission.xacro (robot description, xacro)
@@ -1,5 +1,5 @@
 <?xml version="1.0"?>
 <!--
-  Copyright (c) 2011-2013, PAL Robotics, S.L.
+  Copyright (c) 2011-2014, PAL Robotics, S.L.
   All rights reserved.
   This work is licensed under the Creative Commons Attribution-NonCommercial-NoDerivs 3.0 Unported License.

File: reem_description/urdf/arm/arm.urdf.xacro (robot description, xacro)
@@ -1,5 +1,5 @@
 <?xml version="1.0"?>
 <!--
-  Copyright (c) 2011-2013, PAL Robotics, S.L.
+  Copyright (c) 2011-2014, PAL Robotics, S.L.
   All rights reserved.
   This work is licensed under the Creative Commons Attribution-NonCommercial-NoDerivs 3.0 Unported License.
@@ -9,7 +9,7 @@
 <robot xmlns:xacro="http://ros.org/wiki/xacro">
   <!--File includes-->
-  <include filename="$(find reem_description)/urdf/deg_to_rad.xacro" />
-  <include filename="$(find reem_description)/urdf/arm/wrist.urdf.xacro" />
-  <include filename="$(find reem_description)/urdf/arm/arm.transmission.xacro" />
+  <xacro:include filename="$(find reem_description)/urdf/deg_to_rad.xacro" />
+  <xacro:include filename="$(find reem_description)/urdf/arm/wrist.urdf.xacro" />
+  <xacro:include filename="$(find reem_description)/urdf/arm/arm.transmission.xacro" />
   <!--Constant parameters-->
   <xacro:property name="arm_friction"       value="1.0" />
@@ -158,5 +158,5 @@
       <safety_controller k_position="20"
                          k_velocity="20"
-                         soft_lower_limit="${0.0 * deg_to_rad    + arm_eps}"
+                         soft_lower_limit="${0.0 * deg_to_rad}"
                          soft_upper_limit="${ 130.0 * deg_to_rad - arm_eps}" />
     </joint>

File: reem_description/urdf/arm/wrist.transmission.xacro (robot description, xacro)
@@ -1,5 +1,5 @@
 <?xml version="1.0"?>
 <!--
-  Copyright (c) 2011-2013, PAL Robotics, S.L.
+  Copyright (c) 2011-2014, PAL Robotics, S.L.
   All rights reserved.
   This work is licensed under the Creative Commons Attribution-NonCommercial-NoDerivs 3.0 Unported License.

File: reem_description/urdf/arm/wrist.urdf.xacro (robot description, xacro)
@@ -1,5 +1,5 @@
 <?xml version="1.0"?>
 <!--
-  Copyright (c) 2011-2013, PAL Robotics, S.L.
+  Copyright (c) 2011-2014, PAL Robotics, S.L.
   All rights reserved.
   This work is licensed under the Creative Commons Attribution-NonCommercial-NoDerivs 3.0 Unported License.
@@ -9,6 +9,6 @@
 <robot xmlns:xacro="http://ros.org/wiki/xacro">
   <!--File includes-->
-  <include filename="$(find reem_description)/urdf/deg_to_rad.xacro" />
-  <include filename="$(find reem_description)/urdf/arm/wrist.transmission.xacro" />
+  <xacro:include filename="$(find reem_description)/urdf/deg_to_rad.xacro" />
+  <xacro:include filename="$(find reem_description)/urdf/arm/wrist.transmission.xacro" />
   <!--Constant parameters-->
   <xacro:property name="wrist_friction"     value="1.0" />

File: reem_description/urdf/base/base.gazebo.xacro (robot description, xacro)
@@ -1,5 +1,5 @@
 <?xml version="1.0"?>
 <!--
-  Copyright (c) 2011-2013, PAL Robotics, S.L.
+  Copyright (c) 2011-2014, PAL Robotics, S.L.
   All rights reserved.
   This work is licensed under the Creative Commons Attribution-NonCommercial-NoDerivs 3.0 Unported License.

File: reem_description/urdf/base/base.transmission.xacro (robot description, xacro)
@@ -1,5 +1,5 @@
 <?xml version="1.0"?>
 <!--
-  Copyright (c) 2011-2013, PAL Robotics, S.L.
+  Copyright (c) 2011-2014, PAL Robotics, S.L.
   All rights reserved.
   This work is licensed under the Creative Commons Attribution-NonCommercial-NoDerivs 3.0 Unported License.

File: reem_description/urdf/base/base.urdf.xacro (robot description, xacro)
@@ -1,5 +1,5 @@
 <?xml version="1.0"?>
 <!--
-  Copyright (c) 2011-2013, PAL Robotics, S.L.
+  Copyright (c) 2011-2014, PAL Robotics, S.L.
   All rights reserved.
   This work is licensed under the Creative Commons Attribution-NonCommercial-NoDerivs 3.0 Unported License.
@@ -8,20 +8,17 @@
 -->
 <robot xmlns:xacro="http://ros.org/wiki/xacro">
-  <include filename="$(find reem_description)/urdf/deg_to_rad.xacro" />
-  <include filename="$(find reem_description)/urdf/base/base.gazebo.xacro" />
-  <include filename="$(find reem_description)/urdf/base/base.transmission.xacro" />
-  <include filename="$(find reem_description)/urdf/sensors/sick_laser_reem.urdf.xacro" />
-  <include filename="$(find reem_description)/urdf/sensors/range.urdf.xacro" />
-  <include filename="$(find reem_description)/urdf/sensors/hokuyo_laser_reem.urdf.xacro" />
-  <!-- <include filename="$(find reem_description)/urdf/sensors/microinfinity_xa3300.urdf.xacro" /> -->
-  <!-- <include filename="$(find reem_description)/urdf/sensors/microstrain_3dmgx2_imu.urdf.xacro" /> -->
-  <include filename="$(find reem_description)/urdf/sensors/imu.urdf.xacro"/>
-  <!--include filename="$(find reem_description)/urdf/sensors/hector_imu.urdf.xacro"/-->
-  <include filename="$(find reem_description)/urdf/sensors/bumper.urdf.xacro" />
+  <xacro:include filename="$(find reem_description)/urdf/deg_to_rad.xacro" />
+  <xacro:include filename="$(find reem_description)/urdf/base/base.gazebo.xacro" />
+  <xacro:include filename="$(find reem_description)/urdf/base/base.transmission.xacro" />
+  <xacro:include filename="$(find reem_description)/urdf/sensors/sick_laser_reem.urdf.xacro" />
+  <xacro:include filename="$(find reem_description)/urdf/sensors/range.urdf.xacro" />
+  <xacro:include filename="$(find reem_description)/urdf/sensors/hokuyo_laser_reem.urdf.xacro" />
+  <xacro:include filename="$(find reem_description)/urdf/sensors/imu.urdf.xacro"/>
+  <xacro:include filename="$(find reem_description)/urdf/sensors/bumper.urdf.xacro" />
   <!--wheel characteristics-->
   <property name="dist_between_wheels" value="0.540" />
   <property name="wheel_radius" value="0.093" />
   <property name="wheel_width" value="0.044" />
-  <property name="wheel_torque" value="5.0" />
+  <property name="wheel_torque" value="50.0" />
   <property name="wheel_velocity" value="1.5" /> <!-- m/s -->
  <!--caster characteristics-->
@@ -57,4 +54,15 @@
       </collision>
     </link>
+  <!-- contact model for wheel surface -->
+   <gazebo reference="wheel_${side}_link">
+     <kp>1000000.0</kp>
+     <kd>100.0</kd>
+     <mu1>1.0</mu1>
+     <mu2>1.0</mu2>
+     <fdir1>0 0 1</fdir1>
+     <maxVel>1.0</maxVel>
+     <minDepth>0.00</minDepth>
+     <cfmDamping>1</cfmDamping>
+   </gazebo>
     <joint name="wheel_${side}_joint" type="continuous">
       <parent link="base_link" />
@@ -116,4 +124,15 @@
       </collision>
     </link>
+   <!-- contact model for caster wheel surface -->
+   <gazebo reference="caster_${side}_2_link">
+     <kp>1000000.0</kp>
+     <kd>100.0</kd>
+     <mu1>1.0</mu1>
+     <mu2>1.0</mu2>
+     <fdir1>0 0 1</fdir1>
+     <maxVel>1.0</maxVel>
+     <minDepth>0.00</minDepth>
+     <cfmDamping>1</cfmDamping>
+   </gazebo>
     <joint name="caster_${side}_1_joint" type="continuous">
       <parent link="base_link" />
@@ -262,5 +281,5 @@
    <!-- base sonar -->
     <xacro:range_reem name="${name}_sonar_07" parent="${name}" ros_topic="sonar_base" update_rate="5" maxRange="0.7" minRange="0.01" fov="0.5" radiation="ultrasound">
-      <origin xyz="${-0.48412 -0.0327} 0.15127 0.29" rpy="0.0 0.0 2.6354" />
+      <origin xyz="${-0.48412 + base_link_offset_x} 0.15127 0.29" rpy="0.0 0.0 2.6354" />
     </xacro:range_reem>
    <!-- base sonar -->
@@ -284,9 +303,9 @@
     <!-- bumper front right -->
     <xacro:bumper_reem name="${name}_bumper_01" parent="${name}" ros_topic="bumper_base" update_rate="25" >
-      <origin xyz="${0.325 + base_link_offset_x} -0.15 0.15" rpy="0 0 ${-15.0 * deg_to_rad}" />
+      <origin xyz="${0.225 + base_link_offset_x} -0.15 0.20" rpy="0 0 ${-15.0 * deg_to_rad}" />
     </xacro:bumper_reem>
     <!-- bumper front left -->
     <xacro:bumper_reem name="${name}_bumper_02" parent="${name}" ros_topic="bumper_base" update_rate="25" >
-      <origin xyz="${0.325 + base_link_offset_x} 0.15 0.15" rpy="0 0 ${15.0 * deg_to_rad}" />
+      <origin xyz="${0.225 + base_link_offset_x} 0.15 0.20" rpy="0 0 ${15.0 * deg_to_rad}" />
     </xacro:bumper_reem>
     <!-- bumper left 1 -->
@@ -310,18 +329,8 @@
       <origin xyz="${-0.04 + base_link_offset_x} -0.33 0.1" rpy="0 0 ${-90.0 * deg_to_rad}" />
     </xacro:bumper_reem>
-    <!-- gyroscope microinfinity XA3300
-    <xacro:microinfinity_xa3300 name="imu" parent="${name}" imu_topic="imu/data" update_rate="100.0" stdev="0.0005" >
-        <origin xyz="-0.35231 0.0 0.0040" rpy=" ${180.0 * deg_to_rad} 0 0" />
-    </xacro:microinfinity_xa3300> -->
     <!-- imu -->
-    <xacro:imu name="imu" parent="${name}" topic="imu" update_rate="100.0" stddev="0.00017">
+    <xacro:reem_imu name="base_inclinometer" parent="${name}_link" update_rate="100.0">
       <origin xyz="-0.02977 -0.1497 0.164" rpy="0 ${M_PI} 0"/>
-    </xacro:imu>
-    <!--xacro:microstrain_3dmgx2_imu_v0 name="imu" parent="${name}" imu_topic="imu/data" update_rate="100.0" stdev="0.00017" >
-    <origin xyz="-0.02977 -0.1497 0.164" rpy="0 ${M_PI} 0" />
-    </xacro:microstrain_3dmgx2_imu_v0-->
-    <!--xacro:hector_imu name="imu" parent="${name}" topic="imu" update_rate="100.0" stddev="0.00017">
-      <origin xyz="-0.02977 -0.1497 0.164" rpy="0 ${M_PI} 0"/>
-    </xacro:hector_imu-->
+    </xacro:reem_imu>
     <!-- wheels -->
     <xacro:reem_wheel side="right" reflect="1.0" />
@@ -339,5 +348,5 @@
     <link name="${name}_cargo_link">
       <inertial>
-         <mass value="1.0" />
+        <mass value="1.0" />
         <origin xyz="0 0 0" />
         <inertia ixx="0.01" ixy="0.0" ixz="0.0"
