Commit message: Updating package from local PAL package
- Meshes were updated (bigger hands).
- Some preparation for point_head_action was added.
- Fix warnings (cfmDamping -> implicitSpringDamper) when
  launching model in Gazebo.
- Fix copyright 2014 notes.
- Fix hands mimic joint multiplier for underactuated joints for
  correct transmission.
- Updated footprint.
- base.urdf.xacro crated to simplify launching (I think).
- Added wave and bow motions as example play_motion motions.

File: reem_description/gazebo/gazebo.urdf.xacro (robot description, xacro)
@@ -1,5 +1,5 @@
 <?xml version="1.0"?>
 <!--
-  Copyright (c) 2011-2014, PAL Robotics, S.L.
+  Copyright (c) 2011, PAL Robotics, S.L.
   All rights reserved.
   This work is licensed under the Creative Commons Attribution-NonCommercial-NoDerivs 3.0 Unported License.

File: reem_description/robots/base.urdf.xacro (robot description, xacro)
@@ -1,5 +1,5 @@
 <?xml version="1.0"?>
 <!--
-  Copyright (c) 2013, PAL Robotics, S.L.
+  Copyright (c) 2012, PAL Robotics, S.L.
   All rights reserved.
   This work is licensed under the Creative Commons Attribution-NonCommercial-NoDerivs 3.0 Unported License.
@@ -12,14 +12,12 @@
         xmlns:interface="http://playerstage.sourceforge.net/gazebo/xmlschema/#interface"
         name="reem" >
-  <!-- Stock REEM robot -->
-  <xacro:include filename="$(find reem_description)/robots/reem_full.urdf.xacro" />
-  <!-- PAL printed xtion mount link on top of the head -->
-  <joint name="head_mount_xtion_joint" type="fixed">
-    <origin xyz=" 0.085707 -0.255851  0.0920873 " rpy="1.49965 0.0108274 0.458756"/>
-    <parent link="head_2_link"/>
-    <child link="head_mount_xtion_link"/>
-  </joint>
-  <link name="head_mount_xtion_link">
-    <origin xyz="0.0 0.0 0.0" rpy="0.0 0.0 0.0"/>
-  </link>
+  <!-- The following included files set up definitions of parts of the robot body -->
+  <!-- Base -->
+  <xacro:include filename="$(find reem_description)/urdf/base/base.urdf.xacro" />
+  <!-- Generic simulator_gazebo plugins -->
+<!--   <xacro:include filename="$(find reem_description)/gazebo/gazebo.urdf.xacro" /> -->
+  <!-- Materials for visualization -->
+  <xacro:include filename="$(find reem_description)/urdf/materials.urdf.xacro" />
+  <!-- Base -->
+  <xacro:reem_base  name="base"/>
 </robot>

File: reem_description/robots/reem_arm.urdf.xacro (robot description, xacro)
@@ -1,5 +1,5 @@
 <?xml version="1.0"?>
 <!--
-  Copyright (c) 2012-2014, PAL Robotics, S.L.
+  Copyright (c) 2012, PAL Robotics, S.L.
   All rights reserved.
   This work is licensed under the Creative Commons Attribution-NonCommercial-NoDerivs 3.0 Unported License.

File: reem_description/robots/reem_eye_hand_calibration_left_arm.urdf.xacro (robot description, xacro)
@@ -1,5 +1,5 @@
 <?xml version="1.0"?>
 <!--
-  Copyright (c) 2011-2014, PAL Robotics, S.L.
+  Copyright (c) 2011, PAL Robotics, S.L.
   All rights reserved.
   This work is licensed under the Creative Commons Attribution-NonCommercial-NoDerivs 3.0 Unported License.

File: reem_description/robots/reem_eye_hand_calibration_right_arm.urdf.xacro (robot description, xacro)
@@ -1,5 +1,5 @@
 <?xml version="1.0"?>
 <!--
-  Copyright (c) 2011-2014, PAL Robotics, S.L.
+  Copyright (c) 2013-2014, PAL Robotics, S.L.
   All rights reserved.
   This work is licensed under the Creative Commons Attribution-NonCommercial-NoDerivs 3.0 Unported License.
@@ -12,44 +12,27 @@
         xmlns:interface="http://playerstage.sourceforge.net/gazebo/xmlschema/#interface"
         name="reem" >
-  <!-- The following included files set up definitions of parts of the robot body -->
-  <!-- Base -->
-  <xacro:include filename="$(find reem_description)/urdf/base/base.urdf.xacro" />
-  <!-- Torso -->
-  <xacro:include filename="$(find reem_description)/urdf/torso/torso.urdf.xacro" />
-  <!-- Head -->
-  <xacro:include filename="$(find reem_description)/urdf/head/head.urdf.xacro" />
-  <!-- Arm -->
-  <xacro:include filename="$(find reem_description)/urdf/arm/arm.urdf.xacro" />
-  <!-- Hand -->
-  <xacro:include filename="$(find reem_description)/urdf/hand/hand.urdf.xacro" />
   <!-- Eye-hand calibration chessboard -->
   <xacro:include filename="$(find reem_description)/urdf/eyeHandCalibrationChessBoard.urdf.xacro" />
-  <!-- Camera sensors -->
-  <xacro:include filename="$(find reem_description)/urdf/sensors/stereo_camera.urdf.xacro" />
-<!--   <xacro:include filename="$(find reem_description)/urdf/sensors/back_camera.urdf.xacro" /> -->
-  <!-- Generic simulator_gazebo plugins -->
-  <xacro:include filename="$(find reem_description)/gazebo/gazebo.urdf.xacro" />
-  <!-- Materials for visualization -->
-  <xacro:include filename="$(find reem_description)/urdf/materials.urdf.xacro" />
-  <!-- Now we can start using the macros included above to define the actual robot -->
-  <xacro:reem_base  name="base"/>
-  <xacro:reem_cargo  name="base"/>
-  <xacro:reem_torso name="torso" parent="base_link"/>
-  <xacro:reem_head  name="head"  parent="torso_2_link"/>
-  <!-- The reflect parameter takes the value 1 or -1 to respectively distinguish right from left side in expressions -->
-  <xacro:reem_arm name="arm" parent="torso_2_link" side="right" reflect="1.0"  />
-  <xacro:reem_arm name="arm" parent="torso_2_link" side="left"  reflect="-1.0" />
-  <xacro:reem_hand name="hand" parent="arm_right_tool_link" side="right" reflect="1.0"  />
-  <xacro:reem_hand name="hand" parent="arm_left_tool_link"  side="left"  reflect="-1.0" />
+  <!-- Stock REEM robot -->
+  <xacro:include filename="$(find reem_description)/robots/reem_full.urdf.xacro" />
+  <!-- Head-mounted ASUS Xtion Pro Live -->
+  <xacro:include filename="$(find reem_description)/urdf/sensors/xtion_pro_live.urdf.xacro" />
+  <xacro:xtion_pro_live parent="head_2_link" name="head_mount_xtion" > <!-- name is appended to create link and topic names -->
+     <!-- pose of head_mount_xtion_frame wrt /head_2_link -->
+     <origin xyz="${cal_head_mount_xtion_x}
+                  ${cal_head_mount_xtion_y}
+                  ${cal_head_mount_xtion_z}"
+             rpy="${cal_head_mount_xtion_roll}
+                  ${cal_head_mount_xtion_pitch}
+                  ${cal_head_mount_xtion_yaw}" />
+     <!-- pose of head_mount_xtion_optical_frame wrt head_mount_xtion_frame -->
+     <origin xyz="0.0 0.0 0.0" rpy="-1.57 0.0 -1.57" />
+<!--
+     <property name="M_PI" value="3.1415926535897931" />
+     <origin xyz="0.0 0.0 0.0" rpy="-M_PI/2.0 0.0 -M_PI/2.0" />
+-->
+  </xacro:xtion_pro_live>
+  <!-- Temporaly we will put both right and left checkerboards in the riht hand model -->
   <xacro:reem_eye_hand_calibration_chessboard_gazebo name="eyeHandCalibrationChessBoard" side="right"  reflect="1.0" />
-  <!-- stereo camera -->
-  <!-- IMPORTANT: focal_length = image_width/(2tan(hfov/2)) -->
-  <xacro:stereo_camera_v0 parent="head_2_link" name="stereo" focal_length_left="459.84" hfov_left="71" focal_length_right="459.84" hfov_right="71" image_format="B8G8R8" image_width="656" image_height="492" >
-    <!-- The following transformations expresses the pose of the stereo_link (X pointing forward, Z upwards and Y leftwards, contrary to the stereo_optical_link which has Z pointing forward) wrt  head_2_link. -->
-    <origin xyz="0.08203  -0.09558  0.0365" rpy="1.570796327 0 0" />
-  </xacro:stereo_camera_v0>
-<!--   <xacro:back_camera_v0 parent="torso_2_link" name="back" focal_length="557" hfov="75" image_format="B8G8R8" image_width="640" image_height="480" >  -->
-    <!-- The following transformations expresses the pose of the back_link (X pointing forward, Z upwards and Y leftwards, contrary to the stereo_optical_link which has Z pointing forward) wrt  torso_2_link. -->
-    <!--<origin xyz="-0.140 -0.302 -0.000" rpy="-3.142 1.571 0.211" />
-  </xacro:back_camera_v0>-->
+  <xacro:reem_eye_hand_calibration_chessboard_gazebo name="eyeHandCalibrationChessBoard" side="left"  reflect="-1.0" />
 </robot>

File: reem_description/robots/reem_full.urdf.xacro (robot description, xacro)
@@ -1,5 +1,5 @@
 <?xml version="1.0"?>
 <!--
-  Copyright (c) 2011-2014, PAL Robotics, S.L.
+  Copyright (c) 2011, PAL Robotics, S.L.
   All rights reserved.
   This work is licensed under the Creative Commons Attribution-NonCommercial-NoDerivs 3.0 Unported License.

File: reem_description/robots/reem_head.urdf.xacro (robot description, xacro)
@@ -1,5 +1,5 @@
 <?xml version="1.0"?>
 <!--
-  Copyright (c) 2012-2014, PAL Robotics, S.L.
+  Copyright (c) 2012, PAL Robotics, S.L.
   All rights reserved.
   This work is licensed under the Creative Commons Attribution-NonCommercial-NoDerivs 3.0 Unported License.

File: reem_description/robots/reem_rgbd.urdf.xacro (robot description, xacro)
@@ -1,5 +1,5 @@
 <?xml version="1.0"?>
 <!--
-  Copyright (c) 2013-2014, PAL Robotics, S.L.
+  Copyright (c) 2013, PAL Robotics, S.L.
   All rights reserved.
   This work is licensed under the Creative Commons Attribution-NonCommercial-NoDerivs 3.0 Unported License.

File: reem_description/robots/reem_right_hand_marker.urdf.xacro (robot description, xacro)
@@ -1,5 +1,5 @@
 <?xml version="1.0"?>
 <!--
-  Copyright (c) 2011-2014, PAL Robotics, S.L.
+  Copyright (c) 2011, PAL Robotics, S.L.
   All rights reserved.
   This work is licensed under the Creative Commons Attribution-NonCommercial-NoDerivs 3.0 Unported License.

File: reem_description/robots/reem_torso.urdf.xacro (robot description, xacro)
@@ -1,5 +1,5 @@
 <?xml version="1.0"?>
 <!--
-  Copyright (c) 2012-2014, PAL Robotics, S.L.
+  Copyright (c) 2012, PAL Robotics, S.L.
   All rights reserved.
   This work is licensed under the Creative Commons Attribution-NonCommercial-NoDerivs 3.0 Unported License.

File: reem_description/robots/reem_upper_body.urdf.xacro (robot description, xacro)
@@ -1,5 +1,5 @@
 <?xml version="1.0"?>
 <!--
-  Copyright (c) 2012-2014, PAL Robotics, S.L.
+  Copyright (c) 2012, PAL Robotics, S.L.
   All rights reserved.
   This work is licensed under the Creative Commons Attribution-NonCommercial-NoDerivs 3.0 Unported License.

File: reem_description/robots/reem_wrist.urdf.xacro (robot description, xacro)
@@ -1,5 +1,5 @@
 <?xml version="1.0"?>
 <!--
-  Copyright (c) 2012-2014, PAL Robotics, S.L.
+  Copyright (c) 2012, PAL Robotics, S.L.
   All rights reserved.
   This work is licensed under the Creative Commons Attribution-NonCommercial-NoDerivs 3.0 Unported License.

File: reem_description/urdf/arm/arm.urdf.xacro (robot description, xacro)
@@ -8,5 +8,4 @@
 -->
 <robot xmlns:xacro="http://ros.org/wiki/xacro">
-  <!--File includes-->
   <xacro:include filename="$(find reem_description)/urdf/deg_to_rad.xacro" />
   <xacro:include filename="$(find reem_description)/urdf/arm/wrist.urdf.xacro" />
@@ -174,14 +173,14 @@
    </gazebo>
    <gazebo reference="${name}_${side}_1_joint">
-      <cfmDamping>1</cfmDamping>
+      <implicitSpringDamper>1</implicitSpringDamper>
    </gazebo>
    <gazebo reference="${name}_${side}_2_joint">
-      <cfmDamping>1</cfmDamping>
+      <implicitSpringDamper>1</implicitSpringDamper>
    </gazebo>
    <gazebo reference="${name}_${side}_3_joint">
-      <cfmDamping>1</cfmDamping>
+      <implicitSpringDamper>1</implicitSpringDamper>
    </gazebo>
    <gazebo reference="${name}_${side}_4_joint">
-      <cfmDamping>1</cfmDamping>
+      <implicitSpringDamper>1</implicitSpringDamper>
    </gazebo>
     <!--************************-->

File: reem_description/urdf/arm/wrist.urdf.xacro (robot description, xacro)
@@ -133,11 +133,11 @@
     </gazebo>
     <gazebo reference="${name}_${side}_5_joint">
-        <cfmDamping>1</cfmDamping>
+        <implicitSpringDamper>1</implicitSpringDamper>
     </gazebo>
     <gazebo reference="${name}_${side}_6_joint">
-        <cfmDamping>1</cfmDamping>
+        <implicitSpringDamper>1</implicitSpringDamper>
     </gazebo>
     <gazebo reference="${name}_${side}_7_joint">
-        <cfmDamping>1</cfmDamping>
+        <implicitSpringDamper>1</implicitSpringDamper>
     </gazebo>
     <!-- extensions -->

File: reem_description/urdf/common.xacro (robot description, xacro)
@@ -1,5 +1,5 @@
 <?xml version="1.0"?>
 <!--
-  Copyright (c) 2011-2014, PAL Robotics, S.L.
+  Copyright (c) 2011, PAL Robotics, S.L.
   All rights reserved.
   This work is licensed under the Creative Commons Attribution-NonCommercial-NoDerivs 3.0 Unported License.

File: reem_description/urdf/eyeHandCalibrationChessBoard.urdf.xacro (robot description, xacro)
@@ -1,5 +1,5 @@
 <?xml version="1.0"?>
 <!--
-  Copyright (c) 2011-2014, PAL Robotics, S.L.
+  Copyright (c) 2011, PAL Robotics, S.L.
   All rights reserved.
   This work is licensed under the Creative Commons Attribution-NonCommercial-NoDerivs 3.0 Unported License.
@@ -28,11 +28,10 @@
     </collision>
     <inertial>
-      <mass value="7" />
-      <inertia ixx="0.2333" ixy="0.0" ixz="0.0" iyy="0.2333" iyz="0.0" izz="0.0466" />
+      <mass value="1" />
+      <inertia ixx="0.0001" ixy="0.0" ixz="0.0001" iyy="0.2333" iyz="0.0" izz="0.0001" />
     </inertial>
   </link>
   <gazebo reference="eye_hand_calibration_chessboard_${side}_link">
     <material value="eyeHandCalibrationChessBoard" />
-    <turnGravityOff>false</turnGravityOff>
   </gazebo>
   <joint name="eye_hand_calibration_chessboard_${side}_joint" type="fixed">

File: reem_description/urdf/hand/hand.urdf.xacro (robot description, xacro)
@@ -59,5 +59,5 @@
       <limit lower="${0.0 * deg_to_rad}" upper="${90.0 * deg_to_rad}" effort="2.0" velocity="${hand_max_vel}" />
       <dynamics friction="${hand_friction}" damping="${hand_damping}"/>
-      <mimic joint="${hand_name}_${hand_side}_${finger_name}_joint" multiplier="-1.0" offset="0.0" />
+      <mimic joint="${hand_name}_${hand_side}_${finger_name}_joint" multiplier="${90.0 / 250.0}" offset="0.0" />
     </joint>
     <link name="${hand_name}_${hand_side}_${finger_name}_1_link">
@@ -88,5 +88,5 @@
       <limit lower="${0.0 * deg_to_rad}" upper="${80.0 * deg_to_rad}" effort="1.0" velocity="${hand_max_vel}" />
       <dynamics friction="${hand_friction}" damping="${hand_damping}"/>
-      <mimic joint="${hand_name}_${hand_side}_${finger_name}_joint" multiplier="-1.0" offset="0.0" />
+      <mimic joint="${hand_name}_${hand_side}_${finger_name}_joint" multiplier="${80.0 / 250.0}" offset="0.0" />
     </joint>
     <link name="${hand_name}_${hand_side}_${finger_name}_2_link">
@@ -117,5 +117,5 @@
       <limit lower="${0.0 * deg_to_rad}" upper="${80.0 * deg_to_rad}" effort="1.0" velocity="${hand_max_vel}" />
       <dynamics friction="${hand_friction}" damping="${hand_damping}"/>
-      <mimic joint="${hand_name}_${hand_side}_${finger_name}_joint" multiplier="-1.0" offset="0.0" />
+      <mimic joint="${hand_name}_${hand_side}_${finger_name}_joint" multiplier="${80.0 / 250.0}" offset="0.0" />
     </joint>
     <link name="${hand_name}_${hand_side}_${finger_name}_3_link">
@@ -222,5 +222,5 @@
     </gazebo>
     <gazebo reference="${name}_${side}_thumb_joint">
-       <cfmDamping>1</cfmDamping>
+       <implicitSpringDamper>1</implicitSpringDamper>
     </gazebo>
     <!-- Grasping frame -->

File: reem_description/urdf/head/head.transmission.xacro (robot description, xacro)
@@ -1,5 +1,5 @@
 <?xml version="1.0"?>
 <!--
-  Copyright (c) 2011-2014, PAL Robotics, S.L.
+  Copyright (c) 2011, PAL Robotics, S.L.
   All rights reserved.
   This work is licensed under the Creative Commons Attribution-NonCommercial-NoDerivs 3.0 Unported License.

File: reem_description/urdf/head/head.urdf.xacro (robot description, xacro)
@@ -1,5 +1,5 @@
 <?xml version="1.0"?>
 <!--
-  Copyright (c) 2011-2014, PAL Robotics, S.L.
+  Copyright (c) 2011-2012, PAL Robotics, S.L.
   All rights reserved.
   This work is licensed under the Creative Commons Attribution-NonCommercial-NoDerivs 3.0 Unported License.
@@ -60,5 +60,5 @@
     </gazebo>
     <gazebo reference="${name}_joint">
-       <cfmDamping>1</cfmDamping>
+       <implicitSpringDamper>1</implicitSpringDamper>
     </gazebo>
     <!-- extensions -->
@@ -109,5 +109,5 @@
     </gazebo>
     <gazebo reference="${name}_joint">
-       <cfmDamping>1</cfmDamping>
+       <implicitSpringDamper>1</implicitSpringDamper>
     </gazebo>
     <!-- Head Sonar -->

File: reem_description/urdf/marker/marker.gazebo.xacro (robot description, xacro)
@@ -1,5 +1,5 @@
 <?xml version="1.0"?>
 <!--
-  Copyright (c) 2011-2014, PAL Robotics, S.L.
+  Copyright (c) 2011, PAL Robotics, S.L.
   All rights reserved.
   This work is licensed under the Creative Commons Attribution-NonCommercial-NoDerivs 3.0 Unported License.
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