Commit message: updated capsule_description - big hands

File: reem_description/robots/reem_capsule.urdf.xacro (robot description, xacro)
@@ -14,5 +14,5 @@
   <!-- The following included files set up definitions of parts of the robot body -->
   <!-- Base -->
-  <xacro:include filename="$(find reem_description)/urdf/base/base.urdf.xacro" />
+  <xacro:include filename="$(find reem_description)/urdf/base/base_capsule.urdf.xacro" />
   <!-- Torso -->
   <xacro:include filename="$(find reem_description)/urdf/torso/torso_capsule.urdf.xacro" />

File: reem_description/urdf/arm/arm_capsule.urdf.xacro (robot description, xacro)
@@ -72,7 +72,8 @@
       </visual>
       <collision>
-        <origin xyz="0 0 0" rpy="0 0 0" />
-        <geometry>
-          <mesh filename="package://reem_description/meshes/arm/arm_2_collision.stl" scale="1 1 ${-1*reflect}"/>
+        <origin xyz="0.03 -0.035 0" rpy="${M_PI/2} 0 0" />
+        <geometry>
+		<cylinder length="0.02" radius="0.04" />
+          <!--<mesh filename="package://reem_description/meshes/arm/arm_2_collision.stl" scale="1 1 ${-1*reflect}"/>-->
         </geometry>
       </collision>
@@ -106,8 +107,8 @@
       </visual>
       <collision>
-        <origin xyz="0 0 ${reflect *0.08}" rpy="0 0 0" />
+        <origin xyz="0 0 ${reflect *0.04}" rpy="0 0 0" />
         <geometry>
           <!--<mesh filename="package://reem_description/meshes/arm/arm_3_collision.stl" scale="1 1 ${-1*reflect}"/>-->
-	  <cylinder length="0.18" radius="0.05" />
+	  <cylinder length="0.09" radius="0.05" />
         </geometry>
       </collision>

File: reem_description/urdf/arm/wrist_capsule.urdf.xacro (robot description, xacro)
@@ -107,10 +107,10 @@
       <collision>
         <!-- modified values -->
-        <origin xyz="0 0 ${(0.046 +0.075) * reflect}" rpy="0 0 0" />
+        <origin xyz="0 0 ${(0.046 +0.1) * reflect}" rpy="0 0 0" />
         <!-- original values -->
         <!--<origin xyz="0 0 ${0.046 * 0.75 * reflect}" rpy="0 0 0" />-->
         <geometry>
         <!-- modified values -->
-        <cylinder radius="0.07" length="0.16"/>
+        <cylinder radius="0.13" length="0.04"/>
           <!-- original values -->
           <!--<cylinder radius="0.02" length="0.023"/>-->

File: reem_description/urdf/head/head_capsule.urdf.xacro (robot description, xacro)
@@ -37,7 +37,7 @@
       </visual>
       <collision>
-        <origin xyz="0.0333 0 0.1" rpy="0 0 0" />
+        <origin xyz="0.02 0 0.1" rpy="0 0 0" />
         <geometry>
-	 <cylinder length="0.2" radius="0.15" />
+	 <cylinder length="0.03" radius="0.16" />
           <!--<mesh filename="package://reem_description/meshes/head/head_1_collision.stl"/>-->
         </geometry>

File: reem_description/urdf/torso/torso_capsule.urdf.xacro (robot description, xacro)
@@ -74,5 +74,5 @@
 	<origin xyz="0 -0.16 0" rpy="0 0 0" />
         <geometry>
-	<cylinder length="0.3" radius="0.16" />
+	<cylinder length="0.1" radius="0.16" />
           <!--<mesh filename="package://reem_description/meshes/torso/torso_2_collision.stl" />-->
         </geometry>
