Commit message: setup capsule decomposition inside *_sot.urdf

File: reem_description/robots/reem_upper_body_no_hands.urdf.xacro (robot description, xacro)
@@ -22,28 +22,35 @@
 <!--  <xacro:include filename="$(find reem_description)/urdf/hand/hand.urdf.xacro" />-->
   <!-- Generic simulator_gazebo plugins -->
-  <xacro:include filename="$(find reem_description)/gazebo/gazebo.urdf.xacro" />
+<xacro:include filename="$(find reem_description)/gazebo/gazebo.urdf.xacro" />
   <!-- Materials for visualization -->
-  <xacro:include filename="$(find reem_description)/urdf/materials.urdf.xacro" />
-  <link name="base_link">
-    <inertial>
-      <mass value="50.0" />
-      <origin xyz="0 0 0.1"/>
-      <inertia ixx="1.2083" ixy="0.0" ixz="0.0"
-                iyy="1.2083" iyz="0.0" izz="2.0833" />
-    </inertial>
-    <visual>
-      <origin xyz="0 0 0.1" rpy="0 0 0" />
-      <geometry>
-        <box size="0.5 0.5 0.2" />
-      </geometry>
-      <material name="White" />
-    </visual>
-    <collision>
-      <origin xyz="0 0 0.1" rpy="0 0 0" />
-      <geometry>
-        <box size="0.5 0.5 0.2" />
-      </geometry>
-    </collision>
-  </link>
+<xacro:include filename="$(find reem_description)/urdf/materials.urdf.xacro" />
+    <!--************************-->
+    <!--        BASE            -->
+    <!--************************-->
+    <link name="base_link">
+      <inertial>
+        <origin xyz="-0.14527 -0.00003 0.24721" rpy="0 0 0" /> <!-- assuming d=0.6, w=0.5, h=0.4 -->
+        <mass value="63.58850" />
+        <inertia ixx="3.42"  ixy="0"  ixz="0" iyy="4.33" iyz="0" izz="5.08" /> <!-- assuming d=0.6, w=0.5, h=0.4 -->
+<!--         <origin xyz="-0.15006 -0.00031 0.24965" rpy="0 0 0" /> -->
+<!--         <mass value="64.063" /> -->
+        <!-- NOTE: Assuming box with d=0.6, w=0.5, h=0.4 -->
+<!--         <inertia ixx="3.42"  ixy="0"  ixz="0" iyy="4.33" iyz="0" izz="5.08" /> -->
+      </inertial>
+      <visual>
+        <origin xyz="0 0 0" rpy="0 0 0" />
+        <geometry>
+          <mesh filename="package://reem_description/meshes/base/base.dae" />
+        </geometry>
+        <material name="LightGrey" />
+      </visual>
+      <collision>
+        <origin xyz="0 0 0" rpy="0 0 0" />
+        <geometry>
+          <mesh filename="package://reem_description/meshes/base/base_collision.stl" />
+        </geometry>
+        <material name="LightGrey" />
+      </collision>
+    </link>
   <!-- Body parts -->
   <xacro:reem_torso name="torso" parent="base_link"/>
@@ -52,5 +59,18 @@
   <xacro:reem_arm name="arm" parent="torso_2_link" side="right" reflect="1.0"  />
   <xacro:reem_arm name="arm" parent="torso_2_link" side="left"  reflect="-1.0" />
-  <xacro:reem_hand name="hand" parent="arm_right_tool_link" side="right" reflect="1.0"  />
-  <xacro:reem_hand name="hand" parent="arm_left_tool_link"  side="left"  reflect="-1.0" />
+    <!--************************-->
+    <!--        CAMERA          -->
+    <!--************************-->
+    <link name="camera_link">
+      <inertial>
+        <origin xyz="0.0 0.0 0.0" rpy="0 0 0" />
+        <mass value="0.0" />
+         <inertia ixx="0"  ixy="0"  ixz="0" iyy="0" iyz="0" izz="0" />
+      </inertial>
+    </link>
+    <joint name="camera_joint" type="fixed">
+      <parent link="head_2_link"/>
+      <child link="camera_link"/>
+      <origin xyz="0 0 0" rpy="${180.0 * deg_to_rad} ${-90.0 * deg_to_rad} ${0.0 * deg_to_rad}" />
+    </joint>
 </robot>

Commit message: Add SoT grasping frame

File: reem_description/robots/reem_upper_body_no_hands.urdf.xacro (robot description, xacro)
@@ -20,5 +20,5 @@
   <xacro:include filename="$(find reem_description)/urdf/arm/arm.urdf.xacro" />
   <!-- Hand -->
-<!--  <xacro:include filename="$(find reem_description)/urdf/hand/hand.urdf.xacro" />-->
+  <xacro:include filename="$(find reem_description)/urdf/hand/sot_grasping_frame.urdf.xacro" />
   <!-- Generic simulator_gazebo plugins -->
 <xacro:include filename="$(find reem_description)/gazebo/gazebo.urdf.xacro" />
@@ -59,4 +59,7 @@
   <xacro:reem_arm name="arm" parent="torso_2_link" side="right" reflect="1.0"  />
   <xacro:reem_arm name="arm" parent="torso_2_link" side="left"  reflect="-1.0" />
+  <!-- The reflect parameter takes the value 1 or -1 to respectively distinguish right from left side in expressions -->
+  <xacro:reem_hand name="hand" parent="arm_right_tool_link" side="right" reflect="1.0"  />
+  <xacro:reem_hand name="hand" parent="arm_left_tool_link" side="left"  reflect="-1.0" />
     <!--************************-->
     <!--        CAMERA          -->

File: reem_description/urdf/hand/hand.urdf.xacro (robot description, xacro)
@@ -240,4 +240,20 @@
       </inertial>
     </link>
+    <!-- SOT Grasping frame -->
+    <!-- grasp planner will approach along x-axis -->
+    <joint name="${name}_${side}_sot_grasping_frame_joint" type="fixed">
+      <parent link="${name}_${side}_palm_link" />
+      <child link="${name}_${side}_sot_grasping_frame" />
+      <origin xyz="0.055 ${reflect * 0.054} 0.018" rpy="-0.55 1.54 0" />
+    </joint>
+    <link name="${name}_${side}_sot_grasping_frame">
+      <inertial>
+        <origin xyz="0 0 0" rpy="0 0 0" />
+        <mass value="0.01" /> <!-- matrix below must not be zero, or Gazebo won't load -->
+        <inertia ixx="0.1" ixy="0.0" ixz="0.0"
+                 iyy="0.1" iyz="0.0"
+                 izz="0.1" />
+      </inertial>
+    </link>
     <xacro:hand_thumb_transmission name="${name}_${side}_thumb" reduction="1" />
     <!-- Index finger -->
