Commit message: small hand

File: reem_description/urdf/arm/wrist_capsule.urdf.xacro (robot description, xacro)
@@ -112,5 +112,5 @@
         <geometry>
         <!-- modified values -->
-        <cylinder radius="0.13" length="0.04"/>
+        <cylinder radius="0.10" length="0.04"/>
           <!-- original values -->
           <!--<cylinder radius="0.02" length="0.023"/>-->
